File: boards/VCM_Power/VCM_Power.kicad_sch (KiCad schematic)
At the start: 0 parts

Commit message: Started Power PCB Sheets
Added hierarchal sheets to the Power part of the project. Split the board into separate sections within the schematic project and began adding labels.
Other:
- added sheet 5V Buck Converter (power_5v_buck.kicad_sch)
- added sheet Board Connectors and Power Distribution (connectors_and_dist.kicad_sch)
- added sheet Display 3.3V Supply (display_supply.kicad_sch)
- added sheet Power and Input Protection (power_input_protection.kicad_sch)
- added sheet STM32 3.3 V Supply (stm32_supply.kicad_sch)
