File: boards/VCM_Logic/VCM_Logic.kicad_pcb (KiCad board)
At the start: 2 copper layers, 0 parts

Commit message: Added some documentation, updated main logic sheet
Added a document for information about the chip we will be using. Also added the footprint for the chip to ensure it is the correct one on the logic board project pcb sheet.

Spent some time to create a standards document, there is a pdf for this as well. The idea is to standardize naming and identification of documents such as schematics, pcbs and drawings at least for the VCM but also for the team as a whole if they decide to adopt something more standardized. Began putting together a system descriptions document for the VCM to begin gathering information, specs, etc. all in one place.
Parts:
- added U1: STM32F767ZITx, Package_QFP:LQFP-144_20x20mm_P0.5mm, F.Cu at (150.0, 100.0)
